File: UNOR4Carrier/UNOR4Carrier.kicad_sch (KiCad schematic)
At the start: 1 part, among them IC1 R7FA4M1AB3CFM#AA0

Commit message: wip
Parts:
- added C1, C5: 4.7uF, symbol Device:C
- added C2, C3, C4: 100nF, symbol Device:C
- added R1, R2: 5.1k, symbol Device:R
- added R3: 100k, symbol Device:R
- added R4: 13.7k, symbol Device:R
Connections:
- net GND: now also C1.2, C2.2, C3.2, C4.2, C5.2, R2.2, R4.2
- net +5V: now reaches IC1.11 (VCC_1)
- net +5V: now also IC1.21 (VCC_USB_LDO), IC1.39 (VCC_2), C1.1, C2.1, C3.1, R1.1, R3.1
- net at IC1.16 (P407): now also R1.2, R2.1
- net RESET: now reaches IC1.25 (RES)
- net D8: now reaches IC1.28 (P304)
- net D9: now reaches IC1.29 (P303)
- net D1/TX: now reaches IC1.30 (P302)
- net D0/RX: now reaches IC1.31 (P301)
- net D11/MOSI: now reaches IC1.34 (P109/TDO/SWO)
- net D12/MISO: now reaches IC1.35 (P110/TDI)
- net D13/SCK: now reaches IC1.36 (P111)
- net D10/CS: now reaches IC1.37 (P112)
- net at IC1.4 (VBATT): now also C4.1
- net D7: now reaches IC1.41 (P107)
- net D6: now reaches IC1.42 (P106)
- net D2: now reaches IC1.43 (P105)
- net D3: now reaches IC1.44 (P104)
- net D4: now reaches IC1.45 (P103)
- net D5: now reaches IC1.46 (P102)
- net A4/SDA: now reaches IC1.47 (P101)
- net A5/SCL: now reaches IC1.48 (P100)
- net at IC1.49 (P500): now also R3.2, R4.1
- net at IC1.5 (VCL): now also C5.1
- net A0: now reaches IC1.53 (P014)
- net A3: now reaches IC1.62 (P002)
- net A2: now reaches IC1.63 (P001)
- net A1: now reaches IC1.64 (P000)
- no-connect marks 2 -> 16
Other:
- moved on the sheet: IC1
